Commit message: Trajectory Control - Multi-joint Control

File: src/aaly_urdf/urdf/base_sdf3.urdf.xacro (robot description, xacro)
@@ -1,8 +1,4 @@
 <?xml version="1.0" ?>
 <robot name="aaly">
-  <joint name="fixed" type="floating">
-      <parent link="world"/>
-      <child link="aaly__base_link"/>
-  </joint>
   <joint name="aaly__knee_left_back_joint" type="revolute">
     <parent link="aaly__base_link"/>
@@ -12,8 +8,15 @@
     <limit effort="100.0" lower="0.0" upper="5.23598775598" velocity="1.0"/>
   </joint>
+  <joint name="aaly__leg_left_back_joint" type="fixed">
+    <parent link="aaly__knee_left_back_motor"/>
+    <child link="aaly__leg_left_back"/>
+    <origin rpy="0  0  0" xyz="-0.0035  -0.0159  -0.06587"/>
+    <axis xyz="0  0  0"/>
+    <limit effort="0" lower="0" upper="0" velocity="0"/>
+  </joint>
   <joint name="aaly__thigh_left_back_joint" type="revolute">
-    <parent link="aaly__base_link"/>
-    <child link="aaly__knee_left_back_motor"/>
-    <origin rpy="0  0  0" xyz="-0.107    0.1144   0.12127"/>
+    <parent link="aaly__leg_left_back"/>
+    <child link="aaly__thigh_left_back_motor"/>
+    <origin rpy="3.14159  0       0" xyz="0.0005  -0.0475   0.01586"/>
     <axis xyz="-1  0  0"/>
     <limit effort="100.0" lower="0.0" upper="5.23598775598" velocity="1.0"/>
@@ -26,4 +29,18 @@
     <limit effort="100.0" lower="0.0" upper="5.23598775598" velocity="1.0"/>
   </joint>
+  <joint name="aaly__leg_left_front_joint" type="fixed">
+    <parent link="aaly__knee_left_front_motor"/>
+    <child link="aaly__leg_left_front"/>
+    <origin rpy="0       0      -3.14159" xyz="0       0.0159  -0.04587"/>
+    <axis xyz="0  0  0"/>
+    <limit effort="0" lower="0" upper="0" velocity="0"/>
+  </joint>
+  <joint name="aaly__thigh_left_front_joint" type="revolute">
+    <parent link="aaly__leg_left_front"/>
+    <child link="aaly__thigh_left_front_motor"/>
+    <origin rpy="3.14159  0       3.14159" xyz="0.0005  -0.0475  -0.00413"/>
+    <axis xyz="1  0  0"/>
+    <limit effort="100.0" lower="0.0" upper="5.23598775598" velocity="1.0"/>
+  </joint>
   <joint name="aaly__knee_right_back_joint" type="revolute">
     <parent link="aaly__base_link"/>
@@ -33,4 +50,18 @@
     <limit effort="100.0" lower="0.0" upper="5.23598775598" velocity="1.0"/>
   </joint>
+  <joint name="aaly__leg_right_back_joint" type="fixed">
+    <parent link="aaly__knee_right_back_motor"/>
+    <child link="aaly__leg_right_back"/>
+    <origin rpy="0  0  0" xyz="-0.00024  0.0159  -0.04587"/>
+    <axis xyz="0  0  0"/>
+    <limit effort="0" lower="0" upper="0" velocity="0"/>
+  </joint>
+  <joint name="aaly__thigh_right_back_joint" type="revolute">
+    <parent link="aaly__leg_right_back"/>
+    <child link="aaly__thigh_right_back_motor"/>
+    <origin rpy="3.14159  0       0" xyz="0.0005  0.0475  0"/>
+    <axis xyz="-1  0  0"/>
+    <limit effort="100.0" lower="0.0" upper="5.23598775598" velocity="1.0"/>
+  </joint>
   <joint name="aaly__knee_right_front_joint" type="revolute">
     <parent link="aaly__base_link"/>
@@ -43,7 +74,14 @@
     <parent link="aaly__knee_right_front_motor"/>
     <child link="aaly__leg_right_front"/>
-    <origin rpy="0  0  0" xyz="0     0.034  0"/>
-    <axis xyz="0  0  0"/>
-    <limit effort="0" lower="0" upper="0" velocity="0"/>
+    <origin rpy="0       0      -3.14159" xyz="-0.00376 -0.0159  -0.06587"/>
+    <axis xyz="0  0  0"/>
+    <limit effort="0" lower="0" upper="0" velocity="0"/>
+  </joint>
+  <joint name="aaly__thigh_right_front_joint" type="revolute">
+    <parent link="aaly__leg_right_front"/>
+    <child link="aaly__thigh_right_front_motor"/>
+    <origin rpy="3.14159  0       0" xyz="0.0005   0.0475   0.01586"/>
+    <axis xyz="-1  0  0"/>
+    <limit effort="100.0" lower="0.0" upper="5.23598775598" velocity="1.0"/>
   </joint>
   <joint name="aaly__Left_Track_Side_joint" type="fixed">
@@ -78,5 +116,5 @@
     <parent link="aaly__Left_Side_Track_Support"/>
     <child link="aaly__drum3"/>
-    <origin rpy="1.57079  0       0" xyz="0.14157 -0.038   -0.033"/>
+    <origin rpy="1.57079  0       0" xyz="0.14257 -0.038   -0.033"/>
     <axis xyz="0  0 -1"/>
     <limit effort="0" lower="0" upper="0" velocity="0"/>
@@ -85,5 +123,5 @@
     <parent link="aaly__Right_Side_Track_Support"/>
     <child link="aaly__drum4"/>
-    <origin rpy="1.57079  0       0" xyz="0.14157  0.038   -0.033"/>
+    <origin rpy="1.57079  0       0" xyz="0.14257  0.038   -0.033"/>
     <axis xyz="0  0 -1"/>
     <limit effort="0" lower="0" upper="0" velocity="0"/>
@@ -117,6 +155,4 @@
     <limit effort="0" lower="0" upper="0" velocity="0"/>
   </joint>
-  <!-- Used for fixing robot to Gazebo 'base_link' -->
-  <link name="world"/>
   <link name="aaly__base_link">
     <inertial>
@@ -125,5 +161,5 @@
       <inertia ixx="0.0028086383999999997" ixy="0.0" ixz="0.0" iyy="4.3094400000000005e-05" iyz="0.0" izz="0.0028086383999999997"/>
     </inertial>
-    <collision name="aaly___base_link_collision">
+    <collision name="aaly__base_link_collision">
       <origin rpy="0  0  0" xyz="-0.07     0       0.12427"/>
       <geometry>
@@ -131,8 +167,8 @@
       </geometry>
     </collision>
-    <visual name="aaly___base_link_visual">
+    <visual name="aaly__base_link_visual">
       <origin rpy="0  0  0" xyz="-0.07     0       0.12427"/>
       <geometry>
-        <mesh filename="package://aaly__urdf/meshes/Horizontal_Support_Bar_ASB-512.dae" scale="1.0 1.0 1.0"/>
+        <mesh filename="package://aaly_urdf/meshes/Horizontal_Support_Bar_ASB-512.dae" scale="1.0 1.0 1.0"/>
       </geometry>
     </visual>
@@ -153,5 +189,43 @@
       <origin rpy="0  0  0" xyz="0  0  0"/>
       <geometry>
-        <mesh filename="package://aaly__urdf/meshes/AX12-A_origin_same_as_center_of_mass.stl" scale="1.0 1.0 1.0"/>
+        <mesh filename="package://aaly_urdf/meshes/AX12-A_origin_same_as_center_of_mass.stl" scale="1.0 1.0 1.0"/>
+      </geometry>
+    </visual>
+  </link>
+  <link name="aaly__leg_left_back">
+    <inertial>
+      <mass value="0.05"/>
+      <origin rpy="0  0  0" xyz="0  0  0"/>
+      <inertia ixx="1.7083333333333333e-05" ixy="0.0" ixz="0.0" iyy="1.4683333333333334e-05" iyz="0.0" izz="1.0933333333333333e-05"/>
+    </inertial>
+    <collision name="aaly__leg_left_back_collision">
+      <origin rpy="0  0  0" xyz="0  0  0"/>
+      <geometry>
+        <box size="0.04 0.032 0.050"/>
+      </geometry>
+    </collision>
+    <visual name="aaly__leg_left_back_visual">
+      <origin rpy="0  0  0" xyz="0  0  0"/>
+      <geometry>
+        <mesh filename="package://aaly_urdf/meshes/Leg_Left_Back.stl" scale="1.0 1.0 1.0"/>
+      </geometry>
+    </visual>
+  </link>
+  <link name="aaly__thigh_left_back_motor">
+    <inertial>
+      <mass value="0.05"/>
+      <origin rpy="0  0  0" xyz="0  0  0"/>
+      <inertia ixx="1.7083333333333333e-05" ixy="0.0" ixz="0.0" iyy="1.4683333333333334e-05" iyz="0.0" izz="1.0933333333333333e-05"/>
+    </inertial>
+    <collision name="aaly__thigh_left_back_motor_collision">
+      <origin rpy="0  0  0" xyz="0  0  0"/>
+      <geometry>
+        <box size="0.04 0.032 0.050"/>
+      </geometry>
+    </collision>
+    <visual name="aaly__thigh_left_back_motor_visual">
+      <origin rpy="0  0  0" xyz="0  0  0"/>
+      <geometry>
+        <mesh filename="package://aaly_urdf/meshes/AX12-A_origin_same_as_center_of_mass.stl" scale="1.0 1.0 1.0"/>
       </geometry>
     </visual>
@@ -172,5 +246,43 @@
       <origin rpy="0  0  0" xyz="0  0  0"/>
       <geometry>
-        <mesh filename="package://aaly__urdf/meshes/AX12-A_origin_same_as_center_of_mass.stl" scale="1.0 1.0 1.0"/>
+        <mesh filename="package://aaly_urdf/meshes/AX12-A_origin_same_as_center_of_mass.stl" scale="1.0 1.0 1.0"/>
+      </geometry>
+    </visual>
+  </link>
+  <link name="aaly__leg_left_front">
+    <inertial>
+      <mass value="0.05"/>
+      <origin rpy="0  0  0" xyz="0  0  0"/>
+      <inertia ixx="1.7083333333333333e-05" ixy="0.0" ixz="0.0" iyy="1.4683333333333334e-05" iyz="0.0" izz="1.0933333333333333e-05"/>
+    </inertial>
+    <collision name="aaly__leg_left_front_collision">
+      <origin rpy="0  0  0" xyz="0  0  0"/>
+      <geometry>
+        <box size="0.04 0.032 0.050"/>
+      </geometry>
+    </collision>
+    <visual name="aaly__leg_left_front_visual">
+      <origin rpy="0  0  0" xyz="0  0  0"/>
+      <geometry>
+        <mesh filename="package://aaly_urdf/meshes/Leg_Left_Front.stl" scale="1.0 1.0 1.0"/>
+      </geometry>
+    </visual>
+  </link>
+  <link name="aaly__thigh_left_front_motor">
+    <inertial>
+      <mass value="0.05"/>
+      <origin rpy="0  0  0" xyz="0  0  0"/>
+      <inertia ixx="1.7083333333333333e-05" ixy="0.0" ixz="0.0" iyy="1.4683333333333334e-05" iyz="0.0" izz="1.0933333333333333e-05"/>
+    </inertial>
+    <collision name="aaly__thigh_left_front_motor_collision">
+      <origin rpy="0  0  0" xyz="0  0  0"/>
+      <geometry>
+        <box size="0.04 0.032 0.050"/>
+      </geometry>
+    </collision>
+    <visual name="aaly__thigh_left_front_motor_visual">
+      <origin rpy="0  0  0" xyz="0  0  0"/>
+      <geometry>
+        <mesh filename="package://aaly_urdf/meshes/AX12-A_origin_same_as_center_of_mass.stl" scale="1.0 1.0 1.0"/>
       </geometry>
     </visual>
@@ -191,5 +303,43 @@
       <origin rpy="0  0  0" xyz="0  0  0"/>
       <geometry>
-        <mesh filename="package://aaly__urdf/meshes/AX12-A_origin_same_as_center_of_mass.stl" scale="1.0 1.0 1.0"/>
+        <mesh filename="package://aaly_urdf/meshes/AX12-A_origin_same_as_center_of_mass.stl" scale="1.0 1.0 1.0"/>
+      </geometry>
+    </visual>
+  </link>
+  <link name="aaly__leg_right_back">
+    <inertial>
+      <mass value="0.05"/>
+      <origin rpy="0  0  0" xyz="0  0  0"/>
+      <inertia ixx="1.7083333333333333e-05" ixy="0.0" ixz="0.0" iyy="1.4683333333333334e-05" iyz="0.0" izz="1.0933333333333333e-05"/>
+    </inertial>
+    <collision name="aaly__leg_right_back_collision">
+      <origin rpy="0  0  0" xyz="0  0  0"/>
+      <geometry>
+        <box size="0.04 0.032 0.050"/>
+      </geometry>
+    </collision>
+    <visual name="aaly__leg_right_back_visual">
+      <origin rpy="0  0  0" xyz="0  0  0"/>
+      <geometry>
+        <mesh filename="package://aaly_urdf/meshes/Leg_Right_Back.stl" scale="1.0 1.0 1.0"/>
+      </geometry>
+    </visual>
+  </link>
+  <link name="aaly__thigh_right_back_motor">
+    <inertial>
+      <mass value="0.05"/>
+      <origin rpy="0  0  0" xyz="0  0  0"/>
+      <inertia ixx="1.7083333333333333e-05" ixy="0.0" ixz="0.0" iyy="1.4683333333333334e-05" iyz="0.0" izz="1.0933333333333333e-05"/>
+    </inertial>
+    <collision name="aaly__thigh_right_back_motor_collision">
+      <origin rpy="0  0  0" xyz="0  0  0"/>
+      <geometry>
+        <box size="0.04 0.032 0.050"/>
+      </geometry>
+    </collision>
+    <visual name="aaly__thigh_right_back_motor_visual">
+      <origin rpy="0  0  0" xyz="0  0  0"/>
+      <geometry>
+        <mesh filename="package://aaly_urdf/meshes/AX12-A_origin_same_as_center_of_mass.stl" scale="1.0 1.0 1.0"/>
       </geometry>
     </visual>
@@ -210,5 +360,5 @@
       <origin rpy="0  0  0" xyz="0  0  0"/>
       <geometry>
-        <mesh filename="package://aaly__urdf/meshes/AX12-A_origin_same_as_center_of_mass.stl" scale="1.0 1.0 1.0"/>
+        <mesh filename="package://aaly_urdf/meshes/AX12-A_origin_same_as_center_of_mass.stl" scale="1.0 1.0 1.0"/>
       </geometry>
     </visual>
@@ -229,5 +379,24 @@
       <origin rpy="0  0  0" xyz="0  0  0"/>
       <geometry>
-        <mesh filename="package://aaly__urdf/meshes/Leg_Right_Front.stl" scale="1.0 1.0 1.0"/>
+        <mesh filename="package://aaly_urdf/meshes/Leg_Right_Front.stl" scale="1.0 1.0 1.0"/>
+      </geometry>
+    </visual>
+  </link>
+  <link name="aaly__thigh_right_front_motor">
+    <inertial>
+      <mass value="0.05"/>
+      <origin rpy="0  0  0" xyz="0  0  0"/>
+      <inertia ixx="1.7083333333333333e-05" ixy="0.0" ixz="0.0" iyy="1.4683333333333334e-05" iyz="0.0" izz="1.0933333333333333e-05"/>
+    </inertial>
+    <collision name="aaly__thigh_right_front_motor_collision">
+      <origin rpy="0  0  0" xyz="0  0  0"/>
+      <geometry>
+        <box size="0.04 0.032 0.050"/>
+      </geometry>
+    </collision>
+    <visual name="aaly__thigh_right_front_motor_visual">
+      <origin rpy="0  0  0" xyz="0  0  0"/>
+      <geometry>
+        <mesh filename="package://aaly_urdf/meshes/AX12-A_origin_same_as_center_of_mass.stl" scale="1.0 1.0 1.0"/>
       </geometry>
     </visual>
@@ -239,14 +408,14 @@
       <inertia ixx="1.7083333333333333e-05" ixy="0.0" ixz="0.0" iyy="1.4683333333333334e-05" iyz="0.0" izz="1.0933333333333333e-05"/>
     </inertial>
-    <collision name="aaly___Left_Side_Track_Support_collision">
+    <collision name="aaly__Left_Side_Track_Support_collision">
       <origin rpy="0  0  0" xyz="0     0     0.015"/>
       <geometry>
-        <mesh filename="package://aaly__urdf/meshes/Track_Support_Collision_Mesh.dae" scale="1.0 1.0 1.0"/>
-      </geometry>
-    </collision>
-    <visual name="aaly___Left_Side_Track_Support_visual">
-      <origin rpy="0  0  0" xyz="0  0  0"/>
-      <geometry>
-        <mesh filename="package://aaly__urdf/meshes/Track_Support_Left_Side.dae" scale="1.0 1.0 1.0"/>
+        <mesh filename="package://aaly_urdf/meshes/Track_Support_Collision_Mesh.dae" scale="1.0 1.0 1.0"/>
+      </geometry>
+    </collision>
+    <visual name="aaly__Left_Side_Track_Support_visual">
+      <origin rpy="0  0  0" xyz="0  0  0"/>
+      <geometry>
+        <mesh filename="package://aaly_urdf/meshes/Track_Support_Left_Side.dae" scale="1.0 1.0 1.0"/>
       </geometry>
     </visual>
@@ -258,14 +427,14 @@
       <inertia ixx="1.7083333333333333e-05" ixy="0.0" ixz="0.0" iyy="1.4683333333333334e-05" iyz="0.0" izz="1.0933333333333333e-05"/>
     </inertial>
-    <collision name="aaly___Right_Side_Track_Support_collision">
+    <collision name="aaly__Right_Side_Track_Support_collision">
       <origin rpy="0  0  0" xyz="0     0     0.015"/>
       <geometry>
-        <mesh filename="package://aaly__urdf/meshes/Track_Support_Collision_Mesh.dae" scale="1.0 1.0 1.0"/>
-      </geometry>
-    </collision>
-    <visual name="aaly___Left_Side_Track_Support_visual">
-      <origin rpy="0  0  0" xyz="0  0  0"/>
-      <geometry>
-        <mesh filename="package://aaly__urdf/meshes/Track_Support_Right_Side.dae" scale="1.0 1.0 1.0"/>
+        <mesh filename="package://aaly_urdf/meshes/Track_Support_Collision_Mesh.dae" scale="1.0 1.0 1.0"/>
+      </geometry>
+    </collision>
+    <visual name="aaly__Left_Side_Track_Support_visual">
+      <origin rpy="0  0  0" xyz="0  0  0"/>
+      <geometry>
+        <mesh filename="package://aaly_urdf/meshes/Track_Support_Right_Side.dae" scale="1.0 1.0 1.0"/>
       </geometry>
     </visual>
@@ -277,5 +446,5 @@
       <inertia ixx="4.0003370625000006e-05" ixy="0.0" ixz="0.0" iyy="4.0003370625000006e-05" iyz="0.0" izz="3.624778125000001e-05"/>
     </inertial>
-    <collision name="aaly___drum1_collision">
+    <collision name="aaly__drum1_collision">
       <origin rpy="0  0  0" xyz="0  0  0"/>
       <geometry>
@@ -283,8 +452,8 @@
       </geometry>
     </collision>
-    <visual name="aaly___drum1_visual">
-      <origin rpy="0  0  0" xyz="0  0  0"/>
-      <geometry>
-        <mesh filename="package://aaly__urdf/meshes/Lynx_Sproket6in_Hub13.dae" scale="1.0 1.0 1.0"/>
+    <visual name="aaly__drum1_visual">
+      <origin rpy="0  0  0" xyz="0  0  0"/>
+      <geometry>
+        <mesh filename="package://aaly_urdf/meshes/Lynx_Sproket6in_Hub13.dae" scale="1.0 1.0 1.0"/>
       </geometry>
     </visual>
@@ -296,5 +465,5 @@
       <inertia ixx="4.0003370625000006e-05" ixy="0.0" ixz="0.0" iyy="4.0003370625000006e-05" iyz="0.0" izz="3.624778125000001e-05"/>
     </inertial>
-    <collision name="aaly___drum2_collision">
+    <collision name="aaly__drum2_collision">
       <origin rpy="0  0  0" xyz="0  0  0"/>
       <geometry>
@@ -302,8 +471,8 @@
       </geometry>
     </collision>
-    <visual name="aaly___drum2_visual">
-      <origin rpy="0  0  0" xyz="0  0  0"/>
-      <geometry>
-        <mesh filename="package://aaly__urdf/meshes/Lynx_Sproket6in_Hub13.dae" scale="1.0 1.0 1.0"/>
+    <visual name="aaly__drum2_visual">
+      <origin rpy="0  0  0" xyz="0  0  0"/>
+      <geometry>
+        <mesh filename="package://aaly_urdf/meshes/Lynx_Sproket6in_Hub13.dae" scale="1.0 1.0 1.0"/>
       </geometry>
     </visual>
@@ -315,5 +484,5 @@
       <inertia ixx="5.5414245624999996e-05" ixy="0.0" ixz="0.0" iyy="5.5414245624999996e-05" iyz="0.0" izz="0.000100604296875"/>
     </inertial>
-    <collision name="aaly___drum3_collision">
+    <collision name="aaly__drum3_collision">
       <origin rpy="0  0  0" xyz="0  0  0"/>
       <geometry>
@@ -321,8 +490,8 @@
       </geometry>
     </collision>
-    <visual name="aaly___drum3_visual">
-      <origin rpy="0  0  0" xyz="0  0  0"/>
-      <geometry>
-        <mesh filename="package://aaly__urdf/meshes/Lynx_Sproket9in_Hub13.dae" scale="1.0 1.0 1.0"/>
+    <visual name="aaly__drum3_visual">
+      <origin rpy="0  0  0" xyz="0  0  0"/>
+      <geometry>
+        <mesh filename="package://aaly_urdf/meshes/Lynx_Sproket9in_Hub13.dae" scale="1.0 1.0 1.0"/>
       </geometry>
     </visual>
@@ -334,5 +503,5 @@
       <inertia ixx="5.5414245624999996e-05" ixy="0.0" ixz="0.0" iyy="5.5414245624999996e-05" iyz="0.0" izz="0.000100604296875"/>
     </inertial>
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
Commit message: Adding thighs parts

File: src/aaly_urdf/urdf/base_sdf3.urdf.xacro (robot description, xacro)
@@ -15,5 +15,5 @@
     <limit effort="0" lower="0" upper="0" velocity="0"/>
   </joint>
-  <joint name="aaly__thigh_left_back_joint" type="revolute">
+  <joint name="aaly__thigh_left_back_motor_joint" type="revolute">
     <parent link="aaly__leg_left_back"/>
     <child link="aaly__thigh_left_back_motor"/>
@@ -36,5 +36,5 @@
     <limit effort="0" lower="0" upper="0" velocity="0"/>
   </joint>
-  <joint name="aaly__thigh_left_front_joint" type="revolute">
+  <joint name="aaly__thigh_left_front_motor_joint" type="revolute">
     <parent link="aaly__leg_left_front"/>
     <child link="aaly__thigh_left_front_motor"/>
@@ -57,5 +57,5 @@
     <limit effort="0" lower="0" upper="0" velocity="0"/>
   </joint>
-  <joint name="aaly__thigh_right_back_joint" type="revolute">
+  <joint name="aaly__thigh_right_back_motor_joint" type="revolute">
     <parent link="aaly__leg_right_back"/>
     <child link="aaly__thigh_right_back_motor"/>
@@ -78,5 +78,5 @@
     <limit effort="0" lower="0" upper="0" velocity="0"/>
   </joint>
-  <joint name="aaly__thigh_right_front_joint" type="revolute">
+  <joint name="aaly__thigh_right_front_motor_joint" type="revolute">
     <parent link="aaly__leg_right_front"/>
     <child link="aaly__thigh_right_front_motor"/>
@@ -634,5 +634,5 @@
   <transmission name="tran5">
     <type>transmission_interface/SimpleTransmission</type>
-    <joint name="aaly__thigh_left_back_joint">
+    <joint name="aaly__thigh_left_back_motor_joint">
       <hardwareInterface>hardware_interface/PositionJointInterface</hardwareInterface>
     </joint>
@@ -644,5 +644,5 @@
   <transmission name="tran6">
     <type>transmission_interface/SimpleTransmission</type>
-    <joint name="aaly__thigh_left_front_joint">
+    <joint name="aaly__thigh_left_front_motor_joint">
       <hardwareInterface>hardware_interface/PositionJointInterface</hardwareInterface>
     </joint>
@@ -654,5 +654,5 @@
   <transmission name="tran7">
     <type>transmission_interface/SimpleTransmission</type>
-    <joint name="aaly__thigh_right_back_joint">
+    <joint name="aaly__thigh_right_back_motor_joint">
       <hardwareInterface>hardware_interface/PositionJointInterface</hardwareInterface>
     </joint>
@@ -664,5 +664,5 @@
   <transmission name="tran8">
     <type>transmission_interface/SimpleTransmission</type>
-    <joint name="aaly__thigh_right_front_joint">
+    <joint name="aaly__thigh_right_front_motor_joint">
       <hardwareInterface>hardware_interface/PositionJointInterface</hardwareInterface>
     </joint>
