Commit message: Working @ Body Part - Multiple Joints One Link

File: src/aaly_urdf/urdf/base_sdf4.urdf.xacro (robot description, xacro)
@@ -6,10 +6,10 @@
     <origin rpy="0  0  0" xyz="-0.107    0.1144   0.12127"/>
     <axis xyz="-1  0  0"/>
-    <limit effort="100.0" lower="0.0" upper="5.23598775598" velocity="1.0"/>
+    <limit effort="200.0" lower="0.0" upper="5.23598775598" velocity="1.0"/>
   </joint>
   <joint name="aaly__leg_left_back_joint" type="fixed">
     <parent link="aaly__knee_left_back_motor"/>
     <child link="aaly__leg_left_back"/>
-    <origin rpy="0  0  0" xyz="-0.0035  -0.0159  -0.06587"/>
+    <origin rpy="0  0  0" xyz="-0.0015  -0.0239  -0.05622"/>
     <axis xyz="0  0  0"/>
     <limit effort="0" lower="0" upper="0" velocity="0"/>
@@ -18,28 +18,14 @@
     <parent link="aaly__leg_left_back"/>
     <child link="aaly__thigh_left_back_motor"/>
-    <origin rpy="3.14159  0       0" xyz="0.0005  -0.0475   0.01586"/>
-    <axis xyz="-1  0  0"/>
-    <limit effort="100.0" lower="0.0" upper="5.23598775598" velocity="1.0"/>
-  </joint>
-  <joint name="aaly__thigh_left_back_F3_joint" type="fixed">
+    <origin rpy="3.14159  0       0" xyz="-0.0015  -0.0395   0.00622"/>
+    <axis xyz="1  0  0"/>
+    <limit effort="200.0" lower="0.0" upper="5.23598775598" velocity="1.0"/>
+  </joint>
+  <joint name="aaly__thigh_left_back_joint" type="fixed">
     <parent link="aaly__thigh_left_back_motor"/>
-    <child link="aaly__thigh_left_back_F3"/>
-    <origin rpy="-3.14159  0      -1.57079" xyz="0       0      -0.03872"/>
-    <axis xyz="0  0  0"/>
-    <limit effort="0" lower="0" upper="0" velocity="0"/>
-  </joint>
-  <joint name="aaly__thigh_left_back_joint" type="fixed">
-    <parent link="aaly__thigh_left_back_F3"/>
     <child link="aaly__thigh_left_back"/>
-    <origin rpy="0       0      -1.57079" xyz="-0.001  0     0.023"/>
-    <axis xyz="0  0  0"/>
-    <limit effort="0" lower="0" upper="0" velocity="0"/>
-  </joint>
-  <joint name="aaly__body_back_left_joint" type="revolute">
-    <parent link="aaly__thigh_left_back"/>
-    <child link="aaly__body"/>
-    <origin rpy="0  0  0" xyz="-0.03573  0.00186  0.042"/>
-    <axis xyz="1  0  0"/>
-    <limit effort="10000.0" lower="0.0" upper="5.23598775598" velocity="1.0"/>
+    <origin rpy="-3.14159  0      -1.57079" xyz="0       0.001   -0.03322"/>
+    <axis xyz="0  0  0"/>
+    <limit effort="0" lower="0" upper="0" velocity="0"/>
   </joint>
   <joint name="aaly__knee_left_front_joint" type="revolute">
@@ -48,10 +34,10 @@
     <origin rpy="0       0       3.14159" xyz="-0.034    0.1144   0.12127"/>
     <axis xyz="1  0  0"/>
-    <limit effort="100.0" lower="0.0" upper="5.23598775598" velocity="1.0"/>
+    <limit effort="200.0" lower="0.0" upper="5.23598775598" velocity="1.0"/>
   </joint>
   <joint name="aaly__leg_left_front_joint" type="fixed">
     <parent link="aaly__knee_left_front_motor"/>
     <child link="aaly__leg_left_front"/>
-    <origin rpy="0       0      -3.14159" xyz="0       0.0159  -0.04587"/>
+    <origin rpy="0       0      -3.14159" xyz="-0.00376  0.0239  -0.05622"/>
     <axis xyz="0  0  0"/>
     <limit effort="0" lower="0" upper="0" velocity="0"/>
@@ -60,28 +46,14 @@
     <parent link="aaly__leg_left_front"/>
     <child link="aaly__thigh_left_front_motor"/>
-    <origin rpy="3.14159  0       3.14159" xyz="0.0005  -0.0475  -0.00413"/>
-    <axis xyz="1  0  0"/>
-    <limit effort="100.0" lower="0.0" upper="5.23598775598" velocity="1.0"/>
-  </joint>
-  <joint name="aaly__thigh_left_front_F3_joint" type="fixed">
+    <origin rpy="3.14159  0       3.14159" xyz="-0.00076 -0.0395   0.00622"/>
+    <axis xyz="-1  0  0"/>
+    <limit effort="200.0" lower="0.0" upper="5.23598775598" velocity="1.0"/>
+  </joint>
+  <joint name="aaly__thigh_left_joint" type="fixed">
     <parent link="aaly__thigh_left_front_motor"/>
-    <child link="aaly__thigh_left_front_F3"/>
-    <origin rpy="3.14159  0       1.57079" xyz="0       0      -0.03872"/>
-    <axis xyz="0  0  0"/>
-    <limit effort="0" lower="0" upper="0" velocity="0"/>
-  </joint>
-  <joint name="aaly__thigh_left_joint" type="fixed">
-    <parent link="aaly__thigh_left_front_F3"/>
     <child link="aaly__thigh_left_front"/>
-    <origin rpy="0       0      -1.57079" xyz="-0.001  0     0.023"/>
-    <axis xyz="0  0  0"/>
-    <limit effort="0" lower="0" upper="0" velocity="0"/>
-  </joint>
-  <joint name="aaly__body_front_left_joint" type="revolute">
-    <parent link="aaly__thigh_left_front"/>
-    <child link="aaly__body"/>
-    <origin rpy="0  0  0" xyz="-0.03472  0.00186  0.042"/>
-    <axis xyz="1  0  0"/>
-    <limit effort="10000.0" lower="0.0" upper="5.23598775598" velocity="1.0"/>
+    <origin rpy="3.14159  0       1.57079" xyz="0      -0.001   -0.03322"/>
+    <axis xyz="0  0  0"/>
+    <limit effort="0" lower="0" upper="0" velocity="0"/>
   </joint>
   <joint name="aaly__knee_right_back_joint" type="revolute">
@@ -90,10 +62,10 @@
     <origin rpy="0  0  0" xyz="-0.107   -0.1144   0.12127"/>
     <axis xyz="1  0  0"/>
-    <limit effort="100.0" lower="0.0" upper="5.23598775598" velocity="1.0"/>
+    <limit effort="200.0" lower="0.0" upper="5.23598775598" velocity="1.0"/>
   </joint>
   <joint name="aaly__leg_right_back_joint" type="fixed">
     <parent link="aaly__knee_right_back_motor"/>
     <child link="aaly__leg_right_back"/>
-    <origin rpy="0  0  0" xyz="-0.00024  0.0159  -0.04587"/>
+    <origin rpy="0  0  0" xyz="-0.0015   0.0239  -0.05622"/>
     <axis xyz="0  0  0"/>
     <limit effort="0" lower="0" upper="0" velocity="0"/>
@@ -102,28 +74,14 @@
     <parent link="aaly__leg_right_back"/>
     <child link="aaly__thigh_right_back_motor"/>
-    <origin rpy="3.14159  0       0" xyz="0.0005  0.0475  0"/>
+    <origin rpy="3.14159  0       0" xyz="-0.0015   0.0395   0.00622"/>
     <axis xyz="-1  0  0"/>
-    <limit effort="100.0" lower="0.0" upper="5.23598775598" velocity="1.0"/>
-  </joint>
-  <joint name="aaly__thigh_right_back_F3_joint" type="fixed">
+    <limit effort="200.0" lower="0.0" upper="5.23598775598" velocity="1.0"/>
+  </joint>
+  <joint name="aaly__thigh_right_back_joint" type="fixed">
     <parent link="aaly__thigh_right_back_motor"/>
-    <child link="aaly__thigh_right_back_F3"/>
-    <origin rpy="-3.14159  0      -1.57079" xyz="0       0.0005  -0.03872"/>
-    <axis xyz="0  0  0"/>
-    <limit effort="0" lower="0" upper="0" velocity="0"/>
-  </joint>
-  <joint name="aaly__thigh_right_back_joint" type="fixed">
-    <parent link="aaly__thigh_right_back_F3"/>
     <child link="aaly__thigh_right_back"/>
-    <origin rpy="0       0      -1.57079" xyz="-0.0005  0      0.023"/>
-    <axis xyz="0  0  0"/>
-    <limit effort="0" lower="0" upper="0" velocity="0"/>
-  </joint>
-  <joint name="aaly__body_back_right_joint" type="revolute">
-    <parent link="aaly__thigh_right_back"/>
-    <child link="aaly__body"/>
-    <origin rpy="0  0  0" xyz="-0.03573 -0.00013  0.042"/>
-    <axis xyz="1  0  0"/>
-    <limit effort="10000.0" lower="0.0" upper="5.23598775598" velocity="1.0"/>
+    <origin rpy="3.11859  0      -1.57079" xyz="0       0.001   -0.05622"/>
+    <axis xyz="0  0  0"/>
+    <limit effort="0" lower="0" upper="0" velocity="0"/>
   </joint>
   <joint name="aaly__knee_right_front_joint" type="revolute">
@@ -132,10 +90,10 @@
     <origin rpy="0       0       3.14159" xyz="-0.034   -0.1144   0.12127"/>
     <axis xyz="-1  0  0"/>
-    <limit effort="100.0" lower="0.0" upper="5.23598775598" velocity="1.0"/>
+    <limit effort="200.0" lower="0.0" upper="5.23598775598" velocity="1.0"/>
   </joint>
   <joint name="aaly__leg_right_front_joint" type="fixed">
     <parent link="aaly__knee_right_front_motor"/>
     <child link="aaly__leg_right_front"/>
-    <origin rpy="0       0      -3.14159" xyz="-0.00376 -0.0159  -0.06587"/>
+    <origin rpy="0       0      -3.14159" xyz="-0.00376 -0.0239  -0.05622"/>
     <axis xyz="0  0  0"/>
     <limit effort="0" lower="0" upper="0" velocity="0"/>
@@ -144,19 +102,12 @@
     <parent link="aaly__leg_right_front"/>
     <child link="aaly__thigh_right_front_motor"/>
-    <origin rpy="3.14159  0       0" xyz="0.0005   0.0475   0.01586"/>
+    <origin rpy="3.14159  0       0" xyz="0.0005   0.0395   0.00622"/>
     <axis xyz="-1  0  0"/>
-    <limit effort="100.0" lower="0.0" upper="5.23598775598" velocity="1.0"/>
-  </joint>
-  <joint name="aaly__thigh_right_front_F3_joint" type="fixed">
+    <limit effort="200.0" lower="0.0" upper="5.23598775598" velocity="1.0"/>
+  </joint>
+  <joint name="aaly__thigh_right_joint" type="fixed">
     <parent link="aaly__thigh_right_front_motor"/>
-    <child link="aaly__thigh_right_front_F3"/>
-    <origin rpy="-3.14159  0      -1.57079" xyz="-0.00025  0.0005  -0.03872"/>
-    <axis xyz="0  0  0"/>
-    <limit effort="0" lower="0" upper="0" velocity="0"/>
-  </joint>
-  <joint name="aaly__thigh_right_joint" type="fixed">
-    <parent link="aaly__thigh_right_front_F3"/>
     <child link="aaly__thigh_right_front"/>
-    <origin rpy="0       0      -1.57079" xyz="-0.0005  0      0.023"/>
+    <origin rpy="-3.14159  0      -1.57079" xyz="-0.00025  0.001   -0.03322"/>
     <axis xyz="0  0  0"/>
     <limit effort="0" lower="0" upper="0" velocity="0"/>
@@ -164,70 +115,91 @@
   <joint name="aaly__body_front_right_joint" type="revolute">
     <parent link="aaly__thigh_right_front"/>
-    <child link="aaly__body"/>
-    <origin rpy="0  0  0" xyz="-0.03573 -0.00013  0.042"/>
+    <child link="aaly__body1"/>
+    <origin rpy="0       0      -1.57079" xyz="0      0      0.0655"/>
     <axis xyz="1  0  0"/>
-    <limit effort="10000.0" lower="0.0" upper="5.23598775598" velocity="1.0"/>
+    <limit effort="200.0" lower="-5.23598775598" upper="5.23598775598" velocity="1.0"/>
+  </joint>
+  <joint name="aaly__body_back_right_joint" type="revolute">
+    <parent link="aaly__thigh_right_back"/>
+    <child link="aaly__body2"/>
+    <origin rpy="0       0.023   -1.57079" xyz="0      -0.00097  0.04248"/>
+    <axis xyz="1  0  0"/>
+    <limit effort="200.0" lower="-5.23598775598" upper="5.23598775598" velocity="1.0"/>
+  </joint>
+  <joint name="aaly__body_front_left_joint" type="revolute">
+    <parent link="aaly__thigh_left_front"/>
+    <child link="aaly__body3"/>
+    <origin rpy="0       0      -1.57079" xyz="0.002  -0.001   0.0655"/>
+    <axis xyz="1  0  0"/>
+    <limit effort="200.0" lower="-5.23598775598" upper="5.23598775598" velocity="1.0"/>
+  </joint>
+  <joint name="aaly__body_back_left_joint" type="revolute">
+    <parent link="aaly__thigh_left_back"/>
+    <child link="aaly__body4"/>
+    <origin rpy="0       0      -1.57079" xyz="0.002   0      0.0655"/>
+    <axis xyz="1  0  0"/>
+    <limit effort="200.0" lower="-5.23598775598" upper="5.23598775598" velocity="1.0"/>
+  </joint>
+  <joint name="aaly__Right_Track_Side_joint" type="fixed">
+    <parent link="aaly__base_link"/>
+    <child link="aaly__Right_Side_Track_Support"/>
+    <origin rpy="0  0  0" xyz="-0.07122 -0.15412  0.12835"/>
+    <axis xyz="0  0  0"/>
+    <limit effort="0" lower="0" upper="0" velocity="0"/>
   </joint>
   <joint name="aaly__Left_Track_Side_joint" type="fixed">
     <parent link="aaly__base_link"/>
     <child link="aaly__Left_Side_Track_Support"/>
-    <origin rpy="0  0  0" xyz="-0.01373 -0.15812  0.07062"/>
-    <axis xyz="0  0  0"/>
-    <limit effort="0" lower="0" upper="0" velocity="0"/>
-  </joint>
-  <joint name="aaly__Right_Track_Side_joint" type="fixed">
-    <parent link="aaly__base_link"/>
-    <child link="aaly__Right_Side_Track_Support"/>
-    <origin rpy="0  0  0" xyz="-0.01373  0.15812  0.07062"/>
+    <origin rpy="0  0  0" xyz="-0.07122  0.15412  0.12835"/>
     <axis xyz="0  0  0"/>
     <limit effort="0" lower="0" upper="0" velocity="0"/>
   </joint>
   <joint name="aaly__drum_joint1" type="continuous">
+    <parent link="aaly__Right_Side_Track_Support"/>
+    <child link="aaly__drum1"/>
+    <origin rpy="1.57079  0       0" xyz="-0.05361 -0.042   -0.09835"/>
+    <axis xyz="0  0 -1"/>
+  </joint>
+  <joint name="aaly__drum_joint2" type="continuous">
     <parent link="aaly__Left_Side_Track_Support"/>
-    <child link="aaly__drum1"/>
-    <origin rpy="1.57079  0       0" xyz="-0.1111  -0.038   -0.04062"/>
+    <child link="aaly__drum2"/>
+    <origin rpy="1.57079  0       0" xyz="-0.05361  0.042   -0.09835"/>
     <axis xyz="0  0 -1"/>
   </joint>
-  <joint name="aaly__drum_joint2" type="continuous">
+  <joint name="aaly__drum_joint3" type="continuous">
     <parent link="aaly__Right_Side_Track_Support"/>
-    <child link="aaly__drum2"/>
-    <origin rpy="1.57079  0       0" xyz="-0.1111   0.038   -0.04062"/>
+    <child link="aaly__drum3"/>
+    <origin rpy="1.57079  0       0" xyz="0.20006 -0.042   -0.09073"/>
     <axis xyz="0  0 -1"/>
   </joint>
-  <joint name="aaly__drum_joint3" type="continuous">
+  <joint name="aaly__drum_joint4" type="continuous">
     <parent link="aaly__Left_Side_Track_Support"/>
-    <child link="aaly__drum3"/>
-    <origin rpy="1.57079  0       0" xyz="0.14257 -0.038   -0.033"/>
+    <child link="aaly__drum4"/>
+    <origin rpy="1.57079  0       0" xyz="0.20006  0.042   -0.09073"/>
     <axis xyz="0  0 -1"/>
   </joint>
-  <joint name="aaly__drum_joint4" type="continuous">
+  <joint name="aaly__drum_joint5" type="continuous">
     <parent link="aaly__Right_Side_Track_Support"/>
-    <child link="aaly__drum4"/>
-    <origin rpy="1.57079  0       0" xyz="0.14257  0.038   -0.033"/>
+    <child link="aaly__drum5"/>
+    <origin rpy="1.57079  0       0" xyz="0.02517 -0.042    0.02598"/>
     <axis xyz="0  0 -1"/>
   </joint>
-  <joint name="aaly__drum_joint5" type="continuous">
+  <joint name="aaly__drum_joint6" type="continuous">
     <parent link="aaly__Left_Side_Track_Support"/>
-    <child link="aaly__drum5"/>
-    <origin rpy="1.57079  0       0" xyz="-0.03231 -0.038    0.08371"/>
+    <child link="aaly__drum6"/>
+    <origin rpy="1.57079  0       0" xyz="0.02517  0.042    0.02598"/>
     <axis xyz="0  0 -1"/>
   </joint>
-  <joint name="aaly__drum_joint6" type="continuous">
+  <joint name="aaly__Right_Side_Track_Cover_joint" type="fixed">
     <parent link="aaly__Right_Side_Track_Support"/>
-    <child link="aaly__drum6"/>
-    <origin rpy="1.57079  0       0" xyz="-0.03231  0.038    0.08371"/>
-    <axis xyz="0  0 -1"/>
+    <child link="aaly__Right_Side_Track_Cover"/>
+    <origin rpy="0  0  0" xyz="0.05779 -0.077   -0.06673"/>
+    <axis xyz="0  0  0"/>
+    <limit effort="0" lower="0" upper="0" velocity="0"/>
   </joint>
   <joint name="aaly__Left_Side_Track_Cover_joint" type="fixed">
     <parent link="aaly__Left_Side_Track_Support"/>
     <child link="aaly__Left_Side_Track_Cover"/>
-    <origin rpy="0  0  0" xyz="0.00029 -0.07299 -0.00899"/>
-    <axis xyz="0  0  0"/>
-    <limit effort="0" lower="0" upper="0" velocity="0"/>
-  </joint>
-  <joint name="aaly__Right_Side_Track_Cover_joint" type="fixed">
-    <parent link="aaly__Right_Side_Track_Support"/>
-    <child link="aaly__Right_Side_Track_Cover"/>
-    <origin rpy="0  0  0" xyz="0.00029  0.07299 -0.00899"/>
+    <origin rpy="0  0  0" xyz="0.05779  0.077   -0.06673"/>
     <axis xyz="0  0  0"/>
     <limit effort="0" lower="0" upper="0" velocity="0"/>
@@ -237,5 +209,5 @@
       <mass value="0.36"/>
       <origin rpy="0  0  0" xyz="0  0  0"/>
-      <inertia ixx="0.0028086383999999997" ixy="0.0" ixz="0.0" iyy="4.3094400000000005e-05" iyz="0.0" izz="0.0028086383999999997"/>
+      <inertia ixx="0.002814604013121458" ixy="0.0" ixz="0.0" iyy="7.17760831593746e-05" iyz="0.0" izz="0.0028301708345758957"/>
     </inertial>
     <collision name="aaly__base_link_collision">
@@ -255,6 +227,6 @@
     <inertial>
       <mass value="0.05"/>
-      <origin rpy="0  0  0" xyz="0  0  0"/>
-      <inertia ixx="1.7083333333333333e-05" ixy="0.0" ixz="0.0" iyy="1.4683333333333334e-05" iyz="0.0" izz="1.0933333333333333e-05"/>
+      <origin rpy="0  0  0" xyz="0     0    -0.012"/>
+      <inertia ixx="1.2166047261762851e-05" ixy="0.0" ixz="0.0" iyy="1.4468363602365426e-05" iyz="0.0" izz="7.993829324731787e-06"/>
     </inertial>
     <collision name="aaly__knee_left_back_motor_collision">
@@ -273,28 +245,66 @@
   <link name="aaly__leg_left_back">
     <inertial>
-      <mass value="0.05"/>
-      <origin rpy="0  0  0" xyz="0  0  0"/>
-      <inertia ixx="1.7083333333333333e-05" ixy="0.0" ixz="0.0" iyy="1.4683333333333334e-05" iyz="0.0" izz="1.0933333333333333e-05"/>
+      <mass value="0.04"/>
+      <origin rpy="0  0  0" xyz="0  0  0"/>
+      <inertia ixx="2.69490184257131e-05" ixy="0.0" ixz="0.0" iyy="1.843324918045141e-05" iyz="0.0" izz="3.454538603564566e-05"/>
     </inertial>
     <collision name="aaly__leg_left_back_collision">
       <origin rpy="0  0  0" xyz="0  0  0"/>
       <geometry>
+        <box size="0.04 0.04 0.025"/>
+      </geometry>
+    </collision>
+    <visual name="aaly__leg_left_back_visual">
+      <origin rpy="0  0  0" xyz="0  0  0"/>
+      <geometry>
+        <mesh filename="package://aaly_urdf/meshes/Leg_Left_Back.stl" scale="1.0 1.0 1.0"/>
+      </geometry>
+    </visual>
+  </link>
+  <link name="aaly__thigh_left_back_motor">
+    <inertial>
+      <mass value="0.05"/>
+      <origin rpy="0  0  0" xyz="0     0    -0.012"/>
+      <inertia ixx="1.2166047261762851e-05" ixy="0.0" ixz="0.0" iyy="1.4468363602365426e-05" iyz="0.0" izz="7.993829324731787e-06"/>
+    </inertial>
+    <collision name="aaly__thigh_left_back_motor_collision">
+      <origin rpy="0  0  0" xyz="0  0  0"/>
+      <geometry>
         <box size="0.04 0.032 0.050"/>
       </geometry>
     </collision>
-    <visual name="aaly__leg_left_back_visual">
-      <origin rpy="0  0  0" xyz="0  0  0"/>
-      <geometry>
-        <mesh filename="package://aaly_urdf/meshes/Leg_Left_Back.stl" scale="1.0 1.0 1.0"/>
-      </geometry>
-    </visual>
-  </link>
-  <link name="aaly__thigh_left_back_motor">
-    <inertial>
-      <mass value="0.05"/>
-      <origin rpy="0  0  0" xyz="0  0  0"/>
-      <inertia ixx="1.7083333333333333e-05" ixy="0.0" ixz="0.0" iyy="1.4683333333333334e-05" iyz="0.0" izz="1.0933333333333333e-05"/>
-    </inertial>
-    <collision name="aaly__thigh_left_back_motor_collision">
+    <visual name="aaly__thigh_left_back_motor_visual">
+      <origin rpy="0  0  0" xyz="0  0  0"/>
+      <geometry>
+        <mesh filename="package://aaly_urdf/meshes/AX12-A_origin_same_as_center_of_mass.stl" scale="1.0 1.0 1.0"/>
+      </geometry>
+    </visual>
+  </link>
+  <link name="aaly__thigh_left_back">
+    <inertial>
+      <mass value="0.03"/>
+      <origin rpy="0  0  0" xyz="0  0  0"/>
+      <inertia ixx="2.0103848503359805e-05" ixy="0.0" ixz="0.0" iyy="1.2296884544899207e-05" iyz="0.0" izz="1.2205253512522909e-05"/>
+    </inertial>
+    <collision name="aaly__thigh_left_back_collision">
+      <origin rpy="0  0  0" xyz="0     0     0.023"/>
+      <geometry>
+        <box size="0.04 0.032 0.030"/>
+      </geometry>
+    </collision>
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